File: DE0-Nano_DB25/DE0-Nano_DB25.kicad_pcb (KiCad board)
At the start: 2 copper layers, 110.5 x 48.3 mm, 63 parts, among them M1 4-40, M2 4-40, P1 CONN_20X2, P2 DB25, P3 DB25, U1 74CBTLV3861, U2 74CBTLV3861, U3 74CBTLV3861, U4 74CBTLV3861

Commit message: DE0-Nano_DB25: Initial Version
PCB complete and gerbers generated.

Signed-off-by: Charles Steinkuehler <charles@steinkuehler.net>
Parts:
- added G***: LOGO, LOGO, F.Cu at (142.2, 77.5)
Connections:
- P2 pad : (no net) -> GND
- P3 pad : (no net) -> GND
Other:
- board text added: "Copyright 2016 Charles Steinkuehler Open Source Hardware GPL V3"
- board text added: "DE0-Nano_DB25 Version 1.0"
