File: DE0-Nano_DB25/DE0-Nano_DB25.sch (KiCad schematic (older format))
At the start: 59 parts, among them M1 4-40, M2 4-40

Commit message: DE0-Nano_DB25
Initial PCB placed and routed
Ready for final cleanup and gerber file generation

Signed-off-by: Charles Steinkuehler <charles@steinkuehler.net>
Parts:
- removed LD?: LED, ~, symbol LED
- removed W2, W3: CONN_3, symbol CONN_3
- added C5, C6, C7, C8: 100n, CAPC1608x55N, symbol C
- added LED2: Yellow, OSRAM-LED-0805, symbol LED
- added W2, W3: HEADER_3, pin_strip_3, symbol HEADER_3
- LED1: renamed from LD?; value LED -> Yellow; footprint ~ -> OSRAM-LED-0805; Mfg (none) -> Osram; PartNo (none) -> LY R976-PS-36
- P1: renamed from P?; footprint (none) -> Pin_Socket_20x2; Mfg (none) -> Sullins; PartNo (none) -> SFH11-PBPC-D20-ST-BK
- P2, P3: renamed from J?; footprint (none) -> AMP-5747846; Mfg (none) -> Amp; PartNo (none) -> 5747846-4
- PTC1, PTC2: renamed from PTC?; footprint ~ -> BOURNS-MF-NSMF
- W1: value CONN_3 -> HEADER_3; footprint (none) -> pin_strip_3; symbol CONN_3 -> HEADER_3; Mfg (none) -> Harwin; PartNo (none) -> M20-9990345
- gave numbers to parts that had none: 44
Connections:
- wire segments 253 -> 262
Other:
- moved on the sheet: C1, C2, C3, C4, P2, P3, PTC1, PTC2, R1, R10, R11, R12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

Commit message: DE0-Nano_DB25: Update value field for bus level translators
Change the value field for the bus level translators from the incorrect
LVT family (inherited from the standard KiCAD library) to the correct
CBTD family.

Signed-off-by: Charles Steinkuehler <charles@steinkuehler.net>
Parts:
- U1, U2, U3, U4: value 74CBTLV3861 -> 74CBTD3861
Changed lines of the file:
@@
 LIBS:arduino_shieldsNCL
 LIBS:opendous
+LIBS:DE0-Nano_DB25-cache
 EELAYER 27 0
 EELAYER END
@@
 Sheet 1 1
 Title "DE0-Nano_DB25"
-Date "17 apr 2016"
+Date "19 oct 2016"
 Rev "v1.0"
 Comp ""
@@
 P 4800 1500
 F 0 "U1" H 4900 2100 60  0000 L CNN
-F 1 "74CBTLV3861" H 4820 885 60  0000 L CNN
+F 1 "74CBTD3861" H 4820 885 60  0000 L CNN
 F 2 "SOIC127P1030X265-24N" H 4800 1600 60  0001 C CNN
 F 3 "~" H 4800 1600 60  0000 C CNN
@@
 P 4800 3300
 F 0 "U2" H 4900 3900 60  0000 L CNN
-F 1 "74CBTLV3861" H 4820 2685 60  0000 L CNN
+F 1 "74CBTD3861" H 4820 2685 60  0000 L CNN
 F 2 "SOIC127P1030X265-24N" H 4800 3400 60  0001 C CNN
 F 3 "~" H 4800 3400 60  0000 C CNN
@@
 P 4800 5100
 F 0 "U3" H 4900 5700 60  0000 L CNN
-F 1 "74CBTLV3861" H 4820 4485 60  0000 L CNN
+F 1 "74CBTD3861" H 4820 4485 60  0000 L CNN
 F 2 "SOIC127P1030X265-24N" H 4800 5200 60  0001 C CNN
 F 3 "~" H 4800 5200 60  0000 C CNN
@@
 P 4800 6900
 F 0 "U4" H 4900 7500 60  0000 L CNN
-F 1 "74CBTLV3861" H 4820 6285 60  0000 L CNN
+F 1 "74CBTD3861" H 4820 6285 60  0000 L CNN
 F 2 "SOIC127P1030X265-24N" H 4800 7000 60  0001 C CNN
 F 3 "~" H 4800 7000 60  0000 C CNN
