File: DE0_Nano_50pin/DE0_Nano_50pin.kicad_pcb (KiCad board)
At the start: 2 copper layers, 96 x 68.6 mm, 102 parts, among them M1 4-40, M2 4-40, M3 4-40, M4 4-40, P2 CONN_25X2, P3 CONN_25X2, P4 CONN_25X2

Commit message: Update level translators
Switch to 74CBTD16211 level transators in SOP package

Signed-off-by: Charles Steinkuehler <charles@steinkuehler.net>
Parts:
- added U1: 74CBT16211, SOP63P1035X279-56N, F.Cu at (141.5, 79.0)
- added U2: 74CBT16211, SOP63P1035X279-56N, F.Cu at (141.4, 98.2)
- added U3: 74CBT16211, SOP63P1035X279-56N, F.Cu at (175.3, 116.5)
- R1, R10, R11, R12, R13, R14, R15, R16, R17, R18, R19, R2, R20, R21, R22, R23, R24, R25, R26, R27, R28, R29, R3, R30, R31, R32, R33, R34, R35, R36, R37, R38, R39, R4, R40, R41, R42, R43, R44, R45, R46, R47, R48, R49, R5, R50, R51, R52, R53, R54, R55, R56, R57, R58, R59, R6, R60, R61, R62, R63, R64, R65, R66, R67, R68, R69, R7, R70, R71, R72, R8, R9: value 3.3k -> 4.7k
Connections:
- GPIO0 pad 1: /J1B16 -> (no net)
- GPIO0 pad 10: /J1B9 -> (no net)
- GPIO0 pad 13: /J1B6 -> (no net)
- GPIO0 pad 14: /J1B7 -> (no net)
- GPIO0 pad 15: /J1B4 -> (no net)
- GPIO0 pad 16: /J1B5 -> (no net)
- GPIO0 pad 17: /J1B2 -> (no net)
- GPIO0 pad 18: /J1B3 -> (no net)
- GPIO0 pad 19: /J1B0 -> (no net)
- GPIO0 pad 2: /LED0 -> (no net)
- GPIO0 pad 20: /J1B1 -> (no net)
- GPIO0 pad 21: /J2B16 -> (no net)
- GPIO0 pad 22: /LED1 -> (no net)
- GPIO0 pad 23: /J2B14 -> (no net)
- GPIO0 pad 24: /J2B15 -> (no net)
- GPIO0 pad 25: /J2B12 -> (no net)
- GPIO0 pad 26: /J2B13 -> (no net)
- GPIO0 pad 27: /J2B10 -> (no net)
- GPIO0 pad 28: /J2B11 -> (no net)
- GPIO0 pad 3: /J1B14 -> (no net)
- GPIO0 pad 31: /J2B8 -> (no net)
- GPIO0 pad 32: /J2B9 -> (no net)
- GPIO0 pad 33: /J2B6 -> (no net)
- GPIO0 pad 34: /J2B7 -> (no net)
- GPIO0 pad 35: /J2B4 -> (no net)
- GPIO0 pad 36: /J2B5 -> (no net)
- GPIO0 pad 37: /J2B2 -> (no net)
- GPIO0 pad 38: /J2B3 -> (no net)
- GPIO0 pad 39: /J2B0 -> (no net)
- GPIO0 pad 4: /J1B15 -> (no net)
- GPIO0 pad 40: /J2B1 -> (no net)
- GPIO0 pad 5: /J1B12 -> (no net)
- GPIO0 pad 6: /J1B13 -> (no net)
- GPIO0 pad 7: /J1B10 -> (no net)
- GPIO0 pad 8: /J1B11 -> (no net)
- GPIO0 pad 9: /J1B8 -> (no net)
- GPIO1 pad 1: /J1B16 -> (no net)
- GPIO1 pad 10: /J1B9 -> (no net)
- GPIO1 pad 13: /J1B6 -> (no net)
- GPIO1 pad 14: /J1B7 -> (no net)
- GPIO1 pad 15: /J1B4 -> (no net)
- GPIO1 pad 16: /J1B5 -> (no net)
- GPIO1 pad 17: /J1B2 -> (no net)
- GPIO1 pad 18: /J1B3 -> (no net)
- GPIO1 pad 19: /J1B0 -> (no net)
- GPIO1 pad 2: /LED0 -> (no net)
- GPIO1 pad 20: /J1B1 -> (no net)
- GPIO1 pad 21: /J2B16 -> (no net)
- GPIO1 pad 22: /LED1 -> (no net)
- GPIO1 pad 23: /J2B14 -> (no net)
- GPIO1 pad 24: /J2B15 -> (no net)
- GPIO1 pad 25: /J2B12 -> (no net)
- GPIO1 pad 26: /J2B13 -> (no net)
- GPIO1 pad 27: /J2B10 -> (no net)
- GPIO1 pad 28: /J2B11 -> (no net)
- GPIO1 pad 3: /J1B14 -> (no net)
- GPIO1 pad 31: /J2B8 -> (no net)
- GPIO1 pad 32: /J2B9 -> (no net)
- GPIO1 pad 33: /J2B6 -> (no net)
- GPIO1 pad 34: /J2B7 -> (no net)
- GPIO1 pad 35: /J2B4 -> (no net)
- GPIO1 pad 36: /J2B5 -> (no net)
- GPIO1 pad 37: /J2B2 -> (no net)
- GPIO1 pad 38: /J2B3 -> (no net)
- GPIO1 pad 39: /J2B0 -> (no net)
- GPIO1 pad 4: /J1B15 -> (no net)
- GPIO1 pad 40: /J2B1 -> (no net)
- GPIO1 pad 5: /J1B12 -> (no net)
- GPIO1 pad 6: /J1B13 -> (no net)
- GPIO1 pad 7: /J1B10 -> (no net)
- GPIO1 pad 8: /J1B11 -> (no net)
- GPIO1 pad 9: /J1B8 -> (no net)
- LED1 pad K: /LED0 -> (no net)
- LED2 pad K: /LED1 -> (no net)
