File: CRAMPS/CRAMPS.kicad_pcb (KiCad board)
At the start: 2 copper layers, 99.1 x 99.1 mm, 192 parts, among them M101 PCB_GREEN_RMC, M102 LOGO_OSHW, P101 SOCKET_6_LONG, P102 HEADER_2, P103 HEADER_2, P201 PT_2,5-2-5,0-H, P202 KK-2.54-4W, P203 KK-2.54-4W, P204 KK-2.54-4W, P205 KK-2.54-4W, P206 KK-2.54-4W, P207 KK-2.54-4W, P208 POLOLU_SOCKET, P209 POLOLU_SOCKET, P210 POLOLU_SOCKET, P211 POLOLU_SOCKET, P301 HEADER_2, P302 KK-2.54-2W, P303 HEADER_4X2, P304 HEADER_3X2, P305 HEADER_6, P401 PT_2,5-2-5,0-H, P402 PT_2,5-2-5,0-H, P403 PT_2,5-2-5,0-H, P404 PT_1,5-3-3,5-H, P405 PT_1,5-2-3,5-H, P406 PT_1,5-2-3,5-H, P407 KK-2.54-2W, P408 PT_1,5-2-3,5-H, P409 KK-2.54-2W, P501 HEADER_6, P502 HEADER_6X2, P503 HEADER_4X2, P504 HEADER_4X2, P8 BB_EXP_CONN, P9 BB_EXP_CONN, Q101 2N7002K, Q301 2N7002K, Q302 2N7002K, Q303 2N7002K, Q304 2N7002K, Q305 2N7002K, Q401 IRLB8743PBF, Q402 IRLB8743PBF, Q403 IRLB8743PBF, Q404 DMN2075U, Q405 IRLB8743PBF, Q406 DMN2075U, SW101 SW_PUSH, SW102 SW_PUSH, U201 Pololu, U202 Pololu, U203 Pololu, U204 Pololu, U205 Pololu, U206 Pololu, U301 24C256, U302 74ACT244, U501 74CBTD3861

Commit message: Migrate CRAMPS to Kicad v5
Signed-off-by: Michael Brown <producer@holotronic.dk>
Parts:
- BB101: footprint BeagleBone-Pins -> FlyingBone:BeagleBone-Pins
- C201, C202, C203, C204, C205, C206, C401: footprint c_elec_6.3x7.7 -> walter_smd_cap:c_elec_6.3x7.7
- C301, C302, C402, C403, C404, C405, C406, C407, C501, C502, C503, C504, C505, C506, C507, C508, C509: footprint CAPC1608x55N -> Lindeblom:CAPC1608x55N
- D401, D402, D403, D404, D405, D406: footprint DIOM5127X229N -> Lindeblom:DIOM5127X229N
- F201, F401, F402: footprint Fuse-Loose -> Lindeblom:Fuse-Loose
- FH201, FH401, FH402: footprint Keystone-3568 -> Lindeblom:Keystone-3568
- FID1, FID2, FID3, FID4: footprint FIDUCIAL-060 -> Lindeblom:FIDUCIAL-060
- JP201, JP202, JP203, JP204, JP205, JP206, P304: footprint pin_strip_3x2 -> Lindeblom:pin_strip_3x2
- JP301: footprint pin_strip_2x2 -> Lindeblom:pin_strip_2x2
- JP501, P102, P103, P301: footprint pin_strip_2 -> walter_pin_strip:pin_strip_2
- LD101, LD102, LD301, LD302, LD401, LD402, LD403, LD404, LD405, LD406: footprint OSRAM-LED-0603 -> Lindeblom:OSRAM-LED-0603
- M101: footprint OSHW_logo_2 -> modules_rmc:OSHW_logo_2
- M102: footprint PCB_GREEN_RMC -> modules_rmc:PCB_GREEN_RMC
- P101: footprint pin_strip_6 -> walter_pin_strip:pin_strip_6; moved to F.Cu
- P201, P401, P402, P403: value PT_2,5-2-5,0-H -> VAL**; footprint PT_2,5-2-5,0-H -> Lindeblom:PT_2,5-2-5,0-H
- P202, P203, P204, P205, P206, P207: footprint CONN_KK_2.54_4W -> modules_rmc:CONN_KK_2.54_4W
- P208, P209, P210, P211: footprint Pololu_Socket -> Lindeblom:Pololu_Socket
- P302, P407, P409: footprint CONN_KK_2.54_2W -> modules_rmc:CONN_KK_2.54_2W
- P303, P503, P504: footprint pin_strip_4x2 -> Lindeblom:pin_strip_4x2
- P305, P501: footprint pin_strip_6 -> walter_pin_strip:pin_strip_6
- P404: value PT_1,5-3-3,5-H -> VAL**; footprint PT_1,5-3-3,5-H -> Lindeblom:PT_1,5-3-3,5-H
- P405, P406, P408: value PT_1,5-2-3,5-H -> VAL**; footprint PT_1,5-2-3,5-H -> Lindeblom:PT_1,5-2-3,5-H
- P502: footprint pin_strip_6x2 -> walter_pin_strip:pin_strip_6x2
- P8, P9: footprint P8P9_PinHeader -> FlyingBone:P8P9_PinHeader
- Q101, Q301, Q302, Q303, Q304, Q305, Q404, Q406: footprint SOT23GDS -> Tinkerforge:SOT23GDS
- Q401, Q402, Q403, Q405: footprint TO-220AB_IRF2804_RMC -> modules_rmc:TO-220AB_IRF2804_RMC
- R101, R102, R201, R202, R203, R204, R205, R206, R301, R302, R303, R304, R305, R306, R307, R308, R309, R310, R311, R312, R313, R314, R315, R316, R401, R402, R403, R404, R405, R406, R407, R408, R409, R410, R411, R412, R501, R502, R503, R504, R505, R506, R507, R508, R509, R510, R511, R512, R513, R514, R515, R516, R517, R518: footprint RESC1608x55N -> Lindeblom:RESC1608x55N
- S201, S202, S203, S204, S205, S206, S207, S208, S209, S210, S211, S212, S213, S214, S215, S216, S217, S218, S301, S501: footprint Shunt -> Lindeblom:Shunt
- SW101, SW102: footprint SW_6x6_MULTI -> modules_rmc:SW_6x6_MULTI
- U201, U202, U203, U204, U205, U206: footprint POLOLU -> Lindeblom:POLOLU
- U301: footprint SOIC127P600X175-8AN -> Lindeblom:SOIC127P600X175-8AN
- U302: footprint SOIC127P1032X265-20N -> Lindeblom:SOIC127P1032X265-20N
- U501: footprint SOIC127P1030X265-24N -> Lindeblom:SOIC127P1030X265-24N
Connections:
- P101 pad 2: (no net) -> Net-(P101-Pad2)
- P101 pad 3: (no net) -> Net-(P101-Pad3)
- P101 pad 4: (no net) -> Net-(P101-Pad4)
- P101 pad 5: (no net) -> Net-(P101-Pad5)
- P101 pad 6: (no net) -> Net-(P101-Pad6)
- P402 pad 1: /Mosfet Outputs/Ext_Pwr -> (no net)
- P402 pad 2: DGND -> (no net)
- P8 pad 20: (no net) -> Net-(P8-Pad20)
- P8 pad 21: (no net) -> Net-(P8-Pad21)
- P8 pad 22: (no net) -> Net-(P8-Pad22)
- P8 pad 23: (no net) -> Net-(P8-Pad23)
- P8 pad 24: (no net) -> Net-(P8-Pad24)
- P8 pad 25: (no net) -> Net-(P8-Pad25)
- P8 pad 27: (no net) -> Net-(P8-Pad27)
- P8 pad 28: (no net) -> Net-(P8-Pad28)
- P8 pad 29: (no net) -> Net-(P8-Pad29)
- P8 pad 3: (no net) -> Net-(P8-Pad3)
- P8 pad 30: (no net) -> Net-(P8-Pad30)
- P8 pad 31: (no net) -> Net-(P8-Pad31)
- P8 pad 32: (no net) -> Net-(P8-Pad32)
- P8 pad 33: (no net) -> Net-(P8-Pad33)
- P8 pad 34: (no net) -> Net-(P8-Pad34)
- P8 pad 35: (no net) -> Net-(P8-Pad35)
- P8 pad 36: (no net) -> Net-(P8-Pad36)
- P8 pad 37: (no net) -> Net-(P8-Pad37)
- P8 pad 38: (no net) -> Net-(P8-Pad38)
- P8 pad 39: (no net) -> Net-(P8-Pad39)
- P8 pad 4: (no net) -> Net-(P8-Pad4)
- P8 pad 40: (no net) -> Net-(P8-Pad40)
- P8 pad 41: (no net) -> Net-(P8-Pad41)
- P8 pad 42: (no net) -> Net-(P8-Pad42)
- P8 pad 43: (no net) -> Net-(P8-Pad43)
- P8 pad 44: (no net) -> Net-(P8-Pad44)
- P8 pad 45: (no net) -> Net-(P8-Pad45)
- P8 pad 46: (no net) -> Net-(P8-Pad46)
- P8 pad 5: (no net) -> Net-(P8-Pad5)
- P8 pad 6: (no net) -> Net-(P8-Pad6)
- U301 pad 2: (no net) -> Net-(U301-Pad2)
