File: CRAMPS/CRAMPS.sch (KiCad schematic (older format))
At the start: 15 parts, among them M101 PCB_GREEN_RMC, M102 LOGO_OSHW, P101 SOCKET_6_LONG, P102 HEADER_2, P103 HEADER_2, P8 BB_EXP_CONN, P9 BB_EXP_CONN, Q101 2N7002K, SW101 SW_PUSH, SW102 SW_PUSH

Commit message: Migrate CRAMPS to Kicad v5
Signed-off-by: Michael Brown <producer@holotronic.dk>
Parts:
- BB101: footprint BeagleBone-Pins -> FlyingBone:BeagleBone-Pins; symbol BEAGLEBONE-MTG -> beagleboneblack:BEAGLEBONE-MTG
- LD101, LD102: footprint OSRAM-LED-0603 -> Lindeblom:OSRAM-LED-0603; symbol LED -> m_cramps:LED
- M101: footprint OSHW_logo_2 -> modules_rmc:OSHW_logo_2; symbol PCB_GREEN_RMC -> RMC:PCB_GREEN_RMC
- M102: footprint PCB_GREEN_RMC -> modules_rmc:PCB_GREEN_RMC; symbol LOGO_OSHW -> RMC:LOGO_OSHW
- P101: footprint pin_strip_6 -> walter_pin_strip:pin_strip_6; symbol HEADER_6 -> w_connectors:HEADER_6
- P102, P103: footprint pin_strip_2 -> walter_pin_strip:pin_strip_2; symbol HEADER_2 -> w_connectors:HEADER_2
- P8: footprint P8P9_PinHeader -> FlyingBone:P8P9_PinHeader; symbol BB_EXP_CONN_P8 -> m_cramps:BB_EXP_CONN_P8
- P9: footprint P8P9_PinHeader -> FlyingBone:P8P9_PinHeader; symbol BB_EXP_CONN_P9 -> m_cramps:BB_EXP_CONN_P9
- Q101: footprint SOT23GDS -> Tinkerforge:SOT23GDS; symbol FET_N -> w_device:FET_N
- R101, R102: footprint RESC1608x55N -> Lindeblom:RESC1608x55N; symbol R -> m_cramps:R
- SW101, SW102: footprint SW_6x6_MULTI -> modules_rmc:SW_6x6_MULTI; symbol SW_PUSH -> w_device:SW_PUSH
Changed lines of the file:
@@
-EESchema Schematic File Version 2
-LIBS:power
-LIBS:m_cramps
-LIBS:w_connectors
-LIBS:w_device
-LIBS:w_logic
-LIBS:device
-LIBS:transistors
-LIBS:conn
-LIBS:linear
-LIBS:regul
-LIBS:74xx
-LIBS:cmos4000
-LIBS:adc-dac
-LIBS:memory
-LIBS:xilinx
-LIBS:special
-LIBS:microcontrollers
-LIBS:dsp
-LIBS:microchip
-LIBS:analog_switches
-LIBS:motorola
-LIBS:texas
-LIBS:intel
-LIBS:audio
-LIBS:interface
-LIBS:digital-audio
-LIBS:philips
-LIBS:display
-LIBS:cypress
-LIBS:siliconi
-LIBS:opto
-LIBS:atmel
-LIBS:contrib
-LIBS:valves
-LIBS:RMC
-LIBS:arduino_shieldsNCL
-LIBS:opendous
-LIBS:beaglebone
-LIBS:beagleboneblack
+EESchema Schematic File Version 4
 LIBS:CRAMPS-cache
-EELAYER 27 0
+EELAYER 26 0
 EELAYER END
 $Descr A 11000 8500
@@
 $EndSheet
 $Comp
-L LOGO_OSHW M102
+L RMC:LOGO_OSHW M102
 U 1 1 510E82F9
 P 5250 7550
 F 0 "M102" H 5250 7700 60  0000 C CNN
 F 1 "LOGO_OSHW" H 5250 7450 60  0000 C CNN
-F 2 "PCB_GREEN_RMC" H 5150 7600 60  0001 C CNN
+F 2 "modules_rmc:PCB_GREEN_RMC" H 5150 7600 60  0001 C CNN
 F 3 "" H 5250 7550 60  0001 C CNN
 F 4 "N/A" H 5250 7550 60  0001 C CNN "Mfg"
@@
 STATUS\nLED
 $Comp
-L GND #PWR01
+L power1:GND #PWR01
 U 1 1 50FC24E2
 P 7150 5800
@@
 $EndComp
 $Comp
-L LED LD101
+L m_cramps:LED LD101
 U 1 1 50FC24D8
 P 7150 5100
 F 0 "LD101" V 7075 5100 50  0000 C CNN
 F 1 "Yellow" V 7245 5100 50  0000 C CNN
-F 2 "OSRAM-LED-0603" H 7150 5100 60  0001 C CNN
+F 2 "Lindeblom:OSRAM-LED-0603" H 7150 5100 60  0001 C CNN
 F 3 "" H 7150 5100 60  0001 C CNN
 F 4 "Osram" H 5500 6650 60  0001 C CNN "Mfg"
@@
 $EndComp
 $Comp
-L PCB_GREEN_RMC M101
+L RMC:PCB_GREEN_RMC M101
 U 1 1 523E4D4E
 P 4350 7550
 F 0 "M101" H 4350 7700 60  0000 C CNN
 F 1 "PCB_GREEN_RMC" H 4350 7450 60  0000 C CNN
-F 2 "OSHW_logo_2" H 4350 7550 60  0001 C CNN
+F 2 "modules_rmc:OSHW_logo_2" H 4350 7550 60  0001 C CNN
 F 3 "" H 4350 7550 60  0000 C CNN
 F 4 "N/A" H 4350 7550 60  0001 C CNN "Mfg"
@@
 LED
 $Comp
-L +5V #PWR02
+L power1:+5V #PWR02
 U 1 1 52D057D7
 P 7150 4650
@@
 RESETn
 $Comp
-L GND #PWR03
+L power1:GND #PWR03
 U 1 1 52EECC22
 P 9250 5950
@@
 $EndComp
 $Comp
-L SW_PUSH SW102
+L w_device:SW_PUSH SW102
 U 1 1 52EECC28
 P 9250 5700
 F 0 "SW102" H 9250 5850 50  0000 C CNN
 F 1 "SW_PUSH" H 9250 5620 50  0001 C CNN
-F 2 "SW_6x6_MULTI" H 9250 5700 60  0001 C CNN
+F 2 "modules_rmc:SW_6x6_MULTI" H 9250 5700 60  0001 C CNN
 F 3 "" H 9250 5700 60  0001 C CNN
 F 4 "TE" H 5500 8550 60  0001 C CNN "Mfg"
@@
 DGND
 $Comp
-L PWR_FLAG #FLG04
+L power1:PWR_FLAG #FLG04
 U 1 1 52F146AE
 P 1550 7550
@@
 $EndComp
 $Comp
-L GND #PWR05
+L power1:GND #PWR05
 U 1 1 52F146B4
 P 1550 7650
@@
 NoConn ~ 3350 2200
 $Comp
-L HEADER_2 P103
+L w_connectors:HEADER_2 P103
 U 1 1 532B2BE3
 P 9650 5700
 F 0 "P103" H 9700 5850 60  0000 C CNN
 F 1 "HEADER_2" H 9700 5550 60  0001 C CNN
-F 2 "pin_strip_2" H 9650 5700 60  0001 C CNN
+F 2 "walter_pin_strip:pin_strip_2" H 9650 5700 60  0001 C CNN
 F 3 "" H 9650 5700 60  0000 C CNN
 F 4 "Harwin" H 9650 5700 60  0001 C CNN "Mfg"
@@
 	2850 2250 2750 2250
 Wire Wire Line
-	9250 5850 9250 5950
+	9250 5850 9250 5900
 Connection ~ 9250 5900
 Wire Wire Line
-	9100 5500 9550 5500
+	9100 5500 9250 5500
 Wire Wire Line
 	9250 5500 9250 5550
@@
 PWR_BUT
 $Comp
-L GND #PWR06
+L power1:GND #PWR06
 U 1 1 532B2D45
 P 9250 5150
@@
 $EndComp
 $Comp
-L SW_PUSH SW101
+L w_device:SW_PUSH SW101
 U 1 1 532B2D4D
 P 9250 4900
 F 0 "SW101" H 9250 5050 50  0000 C CNN
 F 1 "SW_PUSH" H 9250 4820 50  0001 C CNN
-F 2 "SW_6x6_MULTI" H 9250 4900 60  0001 C CNN
+F 2 "modules_rmc:SW_6x6_MULTI" H 9250 4900 60  0001 C CNN
 F 3 "" H 9250 4900 60  0001 C CNN
 F 4 "TE" H 5500 7750 60  0001 C CNN "Mfg"
@@
 $EndComp
 $Comp
-L HEADER_2 P102
+L w_connectors:HEADER_2 P102
 U 1 1 532B2D53
 P 9650 4900
 F 0 "P102" H 9700 5050 60  0000 C CNN
 F 1 "HEADER_2" H 9700 4750 60  0001 C CNN
-F 2 "pin_strip_2" H 9650 4900 60  0001 C CNN
+F 2 "walter_pin_strip:pin_strip_2" H 9650 4900 60  0001 C CNN
 F 3 "" H 9650 4900 60  0000 C CNN
 F 4 "Harwin" H 9650 4900 60  0001 C CNN "Mfg"
@@
 $EndComp
 Wire Wire Line
-	9250 5050 9250 5150
+	9250 5050 9250 5100
 Connection ~ 9250 5100
 Wire Wire Line
-	9100 4700 9550 4700
+	9100 4700 9250 4700
 Wire Wire Line
 	9250 4700 9250 4750
@@
 	9550 5100 9550 4950
 $Comp
-L R R101
+L m_cramps:R R101
 U 1 1 532B2DC0
 P 7150 4800
 F 0 "R101" V 7100 4800 50  0000 C CNN
 F 1 "330R" V 7220 4800 50  0000 C CNN
-F 2 "RESC1608x55N" H 7150 4800 60  0001 C CNN
+F 2 "Lindeblom:RESC1608x55N" H 7150 4800 60  0001 C CNN
 F 3 "" H 7150 4800 60  0000 C CNN
 F 4 "Stackpole" H 6450 5350 60  0001 C CNN "Mfg"
@@
 	7150 4700 7150 4650
 $Comp
-L FET_N Q101
+L w_device:FET_N Q101
 U 1 1 532B31E8
 P 7100 5550
 F 0 "Q101" H 7400 5600 70  0000 C CNN
 F 1 "2N7002K" H 7400 5500 60  0000 C CNN
-F 2 "SOT23GDS" H 7100 5550 60  0001 C CNN
+F 2 "Tinkerforge:SOT23GDS" H 7100 5550 60  0001 C CNN
 F 3 "" H 7100 5550 60  0000 C CNN
 F 4 "Diodes Inc." H 7100 5550 60  0001 C CNN "Mfg"
@@
 BB ON\nLED\n
 $Comp
-L GND #PWR07
+L power1:GND #PWR07
 U 1 1 532B4906
 P 8100 5300
@@
 $EndComp
 $Comp
-L LED LD102
+L m_cramps:LED LD102
 U 1 1 532B490E
 P 8100 5100
 F 0 "LD102" V 8025 5100 50  0000 C CNN
 F 1 "Green" V 8195 5100 50  0000 C CNN
-F 2 "OSRAM-LED-0603" H 8100 5100 60  0001 C CNN
+F 2 "Lindeblom:OSRAM-LED-0603" H 8100 5100 60  0001 C CNN
 F 3 "" H 8100 5100 60  0001 C CNN
 F 4 "Osram" H 6450 6650 60  0001 C CNN "Mfg"
@@
 $EndComp
 $Comp
-L R R102
+L m_cramps:R R102
 U 1 1 532B491B
 P 8100 4800
 F 0 "R102" V 8050 4800 50  0000 C CNN
 F 1 "330R" V 8170 4800 50  0000 C CNN
-F 2 "RESC1608x55N" H 8100 4800 60  0001 C CNN
+F 2 "Lindeblom:RESC1608x55N" H 8100 4800 60  0001 C CNN
 F 3 "" H 8100 4800 60  0000 C CNN
 F 4 "Stackpole" H 6450 5350 60  0001 C CNN "Mfg"
@@
 	8100 5000 8100 4900
 $Comp
-L BB_EXP_CONN_P8 P8
+L m_cramps:BB_EXP_CONN_P8 P8
 U 1 1 533029B2
 P 3950 2100
 F 0 "P8" H 3945 3355 60  0000 C CNN
 F 1 "BB_EXP_CONN" H 3950 885 60  0001 C CNN
-F 2 "P8P9_PinHeader" H 3600 900 60  0001 C CNN
+F 2 "FlyingBone:P8P9_PinHeader" H 3600 900 60  0001 C CNN
 F 3 "" H 3600 900 60  0000 C CNN
 F 4 "Major League" H 3950 2100 60  0001 C CNN "Mfg"
@@
 $EndComp
 $Comp
-L BB_EXP_CONN_P9 P9
+L m_cramps:BB_EXP_CONN_P9 P9
 U 1 1 533029C1
 P 3950 4900
 F 0 "P9" H 3945 6155 60  0000 C CNN
 F 1 "BB_EXP_CONN" H 3950 3680 60  0001 C CNN
-F 2 "P8P9_PinHeader" H 3600 3700 60  0001 C CNN
+F 2 "FlyingBone:P8P9_PinHeader" H 3600 3700 60  0001 C CNN
 F 3 "" H 3600 3700 60  0000 C CNN
 F 4 "Major League" H 3950 2100 60  0001 C CNN "Mfg"
@@
 	8100 5200 8100 5300
 $Comp
-L HEADER_6 P101
+L w_connectors:HEADER_6 P101
 U 1 1 5330543C
 P 1350 4250
 F 0 "P101" H 1350 4600 60  0000 C CNN
 F 1 "SOCKET_6_LONG" H 1350 3900 60  0001 C CNN
-F 2 "pin_strip_6" H 1350 4250 60  0001 C CNN
+F 2 "walter_pin_strip:pin_strip_6" H 1350 4250 60  0001 C CNN
 F 3 "" H 1350 4250 60  0000 C CNN
 F 4 "Sparkfun" H 1350 4250 60  0001 C CNN "Mfg"
@@
 $EndComp
 Wire Wire Line
-	1350 6700 1800 6700
-Wire Wire Line
-	1350 7100 1800 7100
+	1350 6700 1600 6700
+Wire Wire Line
+	1350 7100 1600 7100
 Text GLabel 1350 6700 0    50   UnSpc ~ 0
 D3.3V
@@
 BeagleBone Logic supply is always 3.3V
 $Comp
-L PWR_FLAG #FLG08
+L power1:PWR_FLAG #FLG08
 U 1 1 53307816
 P 1800 6600
@@
 	1600 7100 1600 7000
 $Comp
-L +5V #PWR09
+L power1:+5V #PWR09
 U 1 1 53307823
 P 1600 7000
@@
 $EndComp
 $Comp
-L PWR_FLAG #FLG010
+L power1:PWR_FLAG #FLG010
 U 1 1 5330782A
 P 1800 7000
@@
 SYS_5V: Low-current supply\nprovided by BeagleBone PMIC\nActive when BeagleBone is running
 $Comp
-L +3.3V #PWR011
+L power1:+3.3V #PWR011
 U 1 1 5330784E
 P 1600 6600
@@
 NoConn ~ 1450 4500
 $Comp
-L GND #PWR012
+L power1:GND #PWR012
 U 1 1 53318CE2
 P 1600 4100
@@
 	1600 4000 1600 4100
 $Comp
-L +5V #PWR013
+L power1:+5V #PWR013
 U 1 1 53356BF0
 P 8100 4650
@@
 	8100 4700 8100 4650
 $Comp
-L BEAGLEBONE-MTG BB101
+L beagleboneblack:BEAGLEBONE-MTG BB101
 U 1 1 535D6E77
 P 1250 5500
 F 0 "BB101" H 1525 6150 60  0000 C CNN
 F 1 "BeagleBone Black" H 1525 5200 60  0000 C CNN
-F 2 "BeagleBone-Pins" H 1425 6050 60  0001 C CNN
+F 2 "FlyingBone:BeagleBone-Pins" H 1425 6050 60  0001 C CNN
 F 3 "" H 1250 5500 60  0000 C CNN
 F 4 "CircuitCo" H 1250 5500 60  0001 C CNN "Mfg"
@@
 	950  5200 850  5200
 Wire Wire Line
-	850  5200 850  5600
+	850  5200 850  5300
 Wire Wire Line
 	950  5500 850  5500
@@
 Connection ~ 850  5300
 $Comp
-L GND #PWR014
+L power1:GND #PWR014
 U 1 1 535D6F73
 P 850 5600
@@
 Text Notes 5050 5250 0    50   ~ 0
 DIR_W
+Wire Wire Line
+	9250 5900 9250 5950
+Wire Wire Line
+	9250 5500 9550 5500
+Wire Wire Line
+	9250 5100 9250 5150
+Wire Wire Line
+	9250 4700 9550 4700
+Wire Wire Line
+	1600 7100 1800 7100
+Wire Wire Line
+	1600 6700 1800 6700
+Wire Wire Line
+	850  5500 850  5600
+Wire Wire Line
+	850  5400 850  5500
+Wire Wire Line
+	850  5300 850  5400
 $EndSCHEMATC
