File: CRAMPS/con_inputs.sch (KiCad schematic (older format))
At the start: 34 parts, among them P501 HEADER_6, P502 HEADER_6X2, P503 HEADER_4X2, P504 HEADER_4X2, U501 74CBTD3861

Commit message: Migrate CRAMPS to Kicad v5
Signed-off-by: Michael Brown <producer@holotronic.dk>
Parts:
- C501, C502, C503, C504, C505, C506, C507, C508, C509: footprint CAPC1608x55N -> Lindeblom:CAPC1608x55N; symbol C -> m_cramps:C
- JP501: footprint pin_strip_2 -> walter_pin_strip:pin_strip_2; symbol JUMP_MINI -> RMC:JUMP_MINI
- P501: footprint pin_strip_6 -> walter_pin_strip:pin_strip_6; symbol HEADER_6 -> w_connectors:HEADER_6
- P502: footprint pin_strip_6x2 -> walter_pin_strip:pin_strip_6x2; symbol HEADER_6X2 -> w_connectors:HEADER_6x2
- P503, P504: footprint pin_strip_4x2 -> Lindeblom:pin_strip_4x2; symbol HEADER_4X2 -> w_connectors:HEADER_4x2
- R501, R502, R503, R504, R505, R506, R507, R508, R509, R510, R511, R512, R513, R514, R515, R516, R517, R518: footprint RESC1608x55N -> Lindeblom:RESC1608x55N; symbol R -> m_cramps:R
- S501: footprint Shunt -> Lindeblom:Shunt; symbol SHUNT -> m_cramps:Shunt
- U501: footprint SOIC127P1030X265-24N -> Lindeblom:SOIC127P1030X265-24N; symbol 74CBTLV3861 -> m_cramps:74CBTLV3861
