File: CRAMPS/con_outputs.sch (KiCad schematic (older format))
At the start: 50 parts, among them P401 PT_2,5-2-5,0-H, P402 PT_2,5-2-5,0-H, P403 PT_2,5-2-5,0-H, P404 PT_1,5-3-3,5-H, P405 PT_1,5-2-3,5-H, P406 PT_1,5-2-3,5-H, P407 KK-2.54-2W, P408 PT_1,5-2-3,5-H, P409 KK-2.54-2W, Q401 IRLB8743PBF, Q402 IRLB8743PBF, Q403 IRLB8743PBF, Q404 DMN2075U, Q405 IRLB8743PBF, Q406 DMN2075U

Commit message: Migrate CRAMPS to Kicad v5
Signed-off-by: Michael Brown <producer@holotronic.dk>
Parts:
- C401: footprint c_elec_6.3x7.7 -> walter_smd_cap:c_elec_6.3x7.7; symbol CP1 -> CRAMPS-rescue:CP1
- C402, C403, C404, C405, C406, C407: footprint CAPC1608x55N -> Lindeblom:CAPC1608x55N; symbol C -> m_cramps:C
- D401, D402, D403, D404, D405, D406: footprint DIOM5127X229N -> Lindeblom:DIOM5127X229N; symbol DIODE -> m_cramps:DIODE
- F401, F402: footprint Fuse-Loose -> Lindeblom:Fuse-Loose; symbol FUSE-LOOSE -> m_cramps:FUSE-LOOSE
- FH401, FH402: footprint Keystone-3568 -> Lindeblom:Keystone-3568; symbol FUSE-HOLDER -> m_cramps:FUSE-HOLDER
- LD401, LD402, LD403, LD404, LD405, LD406: footprint OSRAM-LED-0603 -> Lindeblom:OSRAM-LED-0603; symbol LED -> m_cramps:LED
- P401, P402, P403: footprint PT_2,5-2-5,0-H -> Lindeblom:PT_2,5-2-5,0-H; symbol HEADER_2 -> w_connectors:HEADER_2
- P404: footprint PT_1,5-3-3,5-H -> Lindeblom:PT_1,5-3-3,5-H; symbol HEADER_3 -> w_connectors:HEADER_3
- P405, P406, P408: footprint PT_1,5-2-3,5-H -> Lindeblom:PT_1,5-2-3,5-H; symbol HEADER_2 -> w_connectors:HEADER_2
- P407, P409: footprint CONN_KK_2.54_2W -> modules_rmc:CONN_KK_2.54_2W; symbol HEADER_2 -> w_connectors:HEADER_2
- Q401, Q402, Q403, Q405: footprint TO-220AB_IRF2804_RMC -> modules_rmc:TO-220AB_IRF2804_RMC; symbol MOSFET_N_RMC -> RMC:MOSFET_N_RMC
- Q404, Q406: footprint SOT23GDS -> Tinkerforge:SOT23GDS; symbol MOS_N -> w_device:MOS_N
- R401, R402, R403, R404, R405, R406, R407, R408, R409, R410, R411, R412: footprint RESC1608x55N -> Lindeblom:RESC1608x55N; symbol R -> m_cramps:R
