File: CRAMPS/e-stop.sch (KiCad schematic (older format))
At the start: 34 parts, among them P301 HEADER_2, P302 KK-2.54-2W, P303 HEADER_4X2, P304 HEADER_3X2, P305 HEADER_6, Q301 2N7002K, Q302 2N7002K, Q303 2N7002K, Q304 2N7002K, Q305 2N7002K, U301 24C256, U302 74ACT244

Commit message: Migrate CRAMPS to Kicad v5
Signed-off-by: Michael Brown <producer@holotronic.dk>
Parts:
- C301, C302: footprint CAPC1608x55N -> Lindeblom:CAPC1608x55N; symbol C -> m_cramps:C
- JP301: footprint pin_strip_2x2 -> Lindeblom:pin_strip_2x2; symbol HEADER_2X2 -> w_connectors:HEADER_2x2
- LD301, LD302: footprint OSRAM-LED-0603 -> Lindeblom:OSRAM-LED-0603; symbol LED -> m_cramps:LED
- P301: footprint pin_strip_2 -> walter_pin_strip:pin_strip_2; symbol HEADER_2 -> w_connectors:HEADER_2
- P302: footprint CONN_KK_2.54_2W -> modules_rmc:CONN_KK_2.54_2W; symbol HEADER_2 -> w_connectors:HEADER_2
- P303: footprint pin_strip_4x2 -> Lindeblom:pin_strip_4x2; symbol HEADER_4X2 -> w_connectors:HEADER_4x2
- P304: footprint pin_strip_3x2 -> Lindeblom:pin_strip_3x2; symbol HEADER_3X2 -> w_connectors:HEADER_3x2
- P305: footprint pin_strip_6 -> walter_pin_strip:pin_strip_6; symbol HEADER_6 -> w_connectors:HEADER_6
- Q301, Q302, Q303, Q304, Q305: footprint SOT23GDS -> Tinkerforge:SOT23GDS; symbol FET_N -> w_device:FET_N
- R301, R302, R303, R304, R305, R306, R307, R308, R309, R310, R311, R312, R313, R314, R315, R316: footprint RESC1608x55N -> Lindeblom:RESC1608x55N; symbol R -> m_cramps:R
- S301: footprint Shunt -> Lindeblom:Shunt; symbol SHUNT -> m_cramps:Shunt
- U301: footprint SOIC127P600X175-8AN -> Lindeblom:SOIC127P600X175-8AN; symbol 24C512 -> m_cramps:24C512
- U302: footprint SOIC127P1032X265-20N -> Lindeblom:SOIC127P1032X265-20N; symbol 74HC244 -> w_logic:74HC244
