File: CRAMPS/steppers.sch (KiCad schematic (older format))
At the start: 55 parts, among them P201 PT_2,5-2-5,0-H, P202 KK-2.54-4W, P203 KK-2.54-4W, P204 KK-2.54-4W, P205 KK-2.54-4W, P206 KK-2.54-4W, P207 KK-2.54-4W, P208 POLOLU_SOCKET, P209 POLOLU_SOCKET, P210 POLOLU_SOCKET, P211 POLOLU_SOCKET, U201 Pololu, U202 Pololu, U203 Pololu, U204 Pololu, U205 Pololu, U206 Pololu

Commit message: Migrate CRAMPS to Kicad v5
Signed-off-by: Michael Brown <producer@holotronic.dk>
Parts:
- C201, C202, C203, C204, C205, C206: footprint c_elec_6.3x7.7 -> walter_smd_cap:c_elec_6.3x7.7; symbol CP1 -> CRAMPS-rescue:CP1
- F201: footprint Fuse-Loose -> Lindeblom:Fuse-Loose; symbol FUSE-LOOSE -> m_cramps:FUSE-LOOSE
- FH201: footprint Keystone-3568 -> Lindeblom:Keystone-3568; symbol FUSE-HOLDER -> m_cramps:FUSE-HOLDER
- JP201, JP202, JP203, JP204, JP205, JP206: footprint pin_strip_3x2 -> Lindeblom:pin_strip_3x2; symbol HEADER_3X2 -> w_connectors:HEADER_3x2
- P201: footprint PT_2,5-2-5,0-H -> Lindeblom:PT_2,5-2-5,0-H; symbol HEADER_2 -> w_connectors:HEADER_2
- P202, P203, P204, P205, P206, P207: footprint CONN_KK_2.54_4W -> modules_rmc:CONN_KK_2.54_4W; symbol HEADER_4 -> w_connectors:HEADER_4
- P208, P209, P210, P211: footprint Pololu_Socket -> Lindeblom:Pololu_Socket; symbol POLOLU_SOCKET -> m_cramps:Pololu_Socket
- R201, R202, R203, R204, R205, R206: footprint RESC1608x55N -> Lindeblom:RESC1608x55N; symbol R -> m_cramps:R
- S201, S202, S203, S204, S205, S206, S207, S208, S209, S210, S211, S212, S213, S214, S215, S216, S217, S218: footprint Shunt -> Lindeblom:Shunt; symbol SHUNT -> m_cramps:Shunt
- U201, U202, U203, U204, U205, U206: footprint POLOLU -> Lindeblom:POLOLU; symbol SM_DRIVER -> m_cramps:SM_Driver
